File: esp32-ds3231-ntp-clock/esp32-ds3231-ntp-clock.kicad_sch (KiCad schematic)
At the start: 55 parts, among them J1 Conn_01x04_Socket, J2 USB_C_Receptacle_USB2.0_14P, Q1 PN2222A, Q2 PN2222A, Q3 PN2222A, Q4 PN2222A, SW1 TS09-63-25-WT-160-SMT-TR, SW2 TS09-63-25-WT-160-SMT-TR, U1 ESP32-S3-WROOM-1, U2 DS3231M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

Commit message: Schematics updated
Parts:
- C1, C10, C3, C7: value C -> 22u
- C2, C4, C5, C6, C8, C9: value C -> 0.1u
- R1, R22, R23, R24, R25, R5, R6: value R -> 10k
- R10, R11, R12, R13, R14, R15, R16, R17, R18, R7, R8, R9: value R -> 330
- R19: value R -> 220
- R2, R3, R4: value R -> 0
- R20, R21: value R -> 4.7k
- R26, R27: value R -> 5k
Changed lines of the file:
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@@
 			)
 		)
-		(property "Value" "R"
+		(property "Value" "330"
 			(at 80.01 259.08 90)
 			(effects
@@
 			)
 		)
-		(property "Value" "C"
+		(property "Value" "22u"
 			(at 331.47 228.5999 0)
 			(effects
@@
 			)
 		)
-		(property "Value" "R"
+		(property "Value" "5k"
 			(at 363.22 154.94 90)
 			(effects
@@
 			)
 		)
-		(property "Value" "R"
+		(property "Value" "4.7k"
 			(at 71.12 179.07 90)
 			(effects
@@
 			)
 		)
-		(property "Value" "R"
+		(property "Value" "330"
 			(at 86.36 246.38 90)
 			(effects
@@
 			)
 		)
-		(property "Value" "R"
+		(property "Value" "330"
 			(at 80.01 248.92 90)
 			(effects
@@
 			)
 		)
-		(property "Value" "C"
+		(property "Value" "22u"
 			(at 375.92 228.5999 0)
 			(effects
@@
 			)
 		)
-		(property "Value" "C"
+		(property "Value" "0.1u"
 			(at 341.63 228.5999 0)
 			(effects
@@
 			)
 		)
-		(property "Value" "C"
+		(property "Value" "0.1u"
 			(at 90.17 58.4199 0)
 			(effects
@@
 			)
 		)
-		(property "Value" "R"
+		(property "Value" "5k"
 			(at 363.22 152.4 90)
 			(effects
@@
 			)
 		)
-		(property "Value" "R"
+		(property "Value" "10k"
 			(at 196.85 165.0999 0)
 			(effects
@@
 			)
 		)
-		(property "Value" "R"
+		(property "Value" "10k"
 			(at 184.15 165.0999 0)
 			(effects
@@
 			)
 		)
-		(property "Value" "R"
+		(property "Value" "330"
 			(at 92.71 254 90)
 			(effects
@@
 			)
 		)
-		(property "Value" "R"
+		(property "Value" "330"
 			(at 195.58 228.6 90)
 			(effects
@@
 			)
 		)
-		(property "Value" "R"
+		(property "Value" "10k"
 			(at 82.55 106.6799 0)
 			(effects
@@
 			)
 		)
-		(property "Value" "C"
+		(property "Value" "0.1u"
 			(at 365.76 228.5999 0)
 			(effects
@@
 			)
 		)
-		(property "Value" "C"
+		(property "Value" "0.1u"
 			(at 83.82 114.2999 0)
 			(effects
@@
 			)
 		)
-		(property "Value" "R"
+		(property "Value" "0"
 			(at 173.99 168.91 90)
 			(effects
@@
 			)
 		)
-		(property "Value" "R"
+		(property "Value" "330"
 			(at 73.66 261.62 90)
 			(effects
@@
 			)
 		)
-		(property "Value" "R"
+		(property "Value" "10k"
 			(at 269.24 171.4499 0)
 			(effects
@@
 			)
 		)
-		(property "Value" "R"
+		(property "Value" "10k"
 			(at 278.13 171.4499 0)
 			(effects
@@
 			)
 		)
-		(property "Value" "C"
+		(property "Value" "0.1u"
 			(at 58.42 180.3399 0)
 			(effects
@@
 			)
 		)
-		(property "Value" "C"
+		(property "Value" "0.1u"
 			(at 92.71 63.5 90)
 			(effects
@@
 			)
 		)
-		(property "Value" "R"
+		(property "Value" "0"
 			(at 173.99 177.8 90)
 			(effects
@@
 			)
 		)
-		(property "Value" "C"
+		(property "Value" "22u"
 			(at 48.26 180.3399 0)
 			(effects
@@
 			)
 		)
-		(property "Value" "R"
+		(property "Value" "10k"
 			(at 190.5 165.0999 0)
 			(effects
@@
 			)
 		)
-		(property "Value" "R"
+		(property "Value" "330"
 			(at 73.66 251.46 90)
 			(effects
@@
 			)
 		)
-		(property "Value" "R"
+		(property "Value" "4.7k"
 			(at 76.2 186.69 90)
 			(effects
@@
 			)
 		)
-		(property "Value" "R"
+		(property "Value" "330"
 			(at 86.36 256.54 90)
 			(effects
@@
 			)
 		)
-		(property "Value" "R"
+		(property "Value" "330"
 			(at 242.57 228.6 90)
 			(effects
@@
 			)
 		)
-		(property "Value" "R"
+		(property "Value" "10k"
 			(at 116.84 55.88 90)
 			(effects
@@
 			)
 		)
-		(property "Value" "R"
+		(property "Value" "0"
 			(at 173.99 186.69 90)
 			(effects
@@
 			)
 		)
-		(property "Value" "C"
+		(property "Value" "22u"
 			(at 80.01 58.4199 0)
 			(effects
@@
 			)
 		)
-		(property "Value" "R"
+		(property "Value" "330"
 			(at 171.45 228.6 90)
 			(effects
@@
 			)
 		)
-		(property "Value" "R"
+		(property "Value" "330"
 			(at 218.44 228.6 90)
 			(effects
@@
 			)
 		)
-		(property "Value" "R"
+		(property "Value" "330"
 			(at 92.71 243.84 90)
 			(effects
@@
 			)
 		)
-		(property "Value" "R"
+		(property "Value" "220"
 			(at 73.66 163.83 90)
 			(effects
